Commit message: - changes

File: src/resources/robot_models/kuka_with_gripper.urdf (robot description, URDF)
Before this commit: robot kuka_iiwa_with_robotiq_gripper, 11 links, 10 joints
Links:
- link base_link: geometry collision cylinder length=0.1 radius=0.1; visual cylinder length=0.1 radius=0.1
- link link_1: geometry collision cylinder length=0.36 radius=0.06; visual cylinder length=0.36 radius=0.06
- link link_2: geometry collision sphere radius=0.07; visual sphere radius=0.07
- link link_3: geometry collision cylinder length=0.42 radius=0.06; visual cylinder length=0.42 radius=0.06
- link link_4: geometry collision sphere radius=0.07; visual sphere radius=0.07
- link link_5: geometry collision cylinder length=0.4 radius=0.05; visual cylinder length=0.4 radius=0.05
- link link_6: geometry collision sphere radius=0.06; visual sphere radius=0.06
- link link_7: geometry collision cylinder length=0.126 radius=0.04; visual cylinder length=0.126 radius=0.04
- link robotiq_85_base_link: geometry collision box size=0.08 0.08 0.138; visual box size=0.08 0.08 0.138
Joints:
- joint joint_a1: limit lower=-2.9668 upper=2.9668 -> lower=-2.9668 upper=2.9668 effort=300 velocity=1.7
- joint joint_a2: limit lower=-2.0942 upper=2.0942 -> lower=-2.0942 upper=2.0942 effort=300 velocity=1.7
- joint joint_a3: limit lower=-2.9668 upper=2.9668 -> lower=-2.9668 upper=2.9668 effort=300 velocity=1.7
- joint joint_a4: limit lower=-2.0942 upper=2.0942 -> lower=-2.0942 upper=2.0942 effort=300 velocity=1.7
- joint joint_a5: limit lower=-2.9668 upper=2.9668 -> lower=-2.9668 upper=2.9668 effort=300 velocity=1.7
- joint joint_a6: limit lower=-2.0942 upper=2.0942 -> lower=-2.0942 upper=2.0942 effort=300 velocity=1.7
- joint joint_a7: limit lower=-3.0541 upper=3.0541 -> lower=-3.0541 upper=3.0541 effort=300 velocity=1.7
