Commit message: - ggccnn2 removal refactor + updated grasping logic to be more resilient to rectangles

File: src/resources/robot_models/iiwa14.urdf (robot description, URDF)
Before this commit: robot iiwa14, 12 links, 11 joints
Links:
- link link_0: geometry collision mesh filename=../kuka_description/meshes/iiwa14/collision/link_0_s.stl; visual mesh filename=../kuka_description/meshes/iiwa14/visual/link_0.stl
- link link_1: geometry collision mesh filename=../kuka_description/meshes/iiwa14/collision/link_1_s.stl; visual mesh filename=../kuka_description/meshes/iiwa14/visual/link_1.stl
- link link_2: geometry collision mesh filename=../kuka_description/meshes/iiwa14/collision/link_2_s.stl; visual mesh filename=../kuka_description/meshes/iiwa14/visual/link_2.stl
- link link_3: geometry collision mesh filename=../kuka_description/meshes/iiwa14/collision/link_3_s.stl; visual mesh filename=../kuka_description/meshes/iiwa14/visual/link_3.stl
- link link_4: geometry collision mesh filename=../kuka_description/meshes/iiwa14/collision/link_4_s.stl; visual mesh filename=../kuka_description/meshes/iiwa14/visual/link_4.stl
- link link_5: geometry collision mesh filename=../kuka_description/meshes/iiwa14/collision/link_5_s.stl; visual mesh filename=../kuka_description/meshes/iiwa14/visual/link_5.stl
- link link_6: geometry collision mesh filename=../kuka_description/meshes/iiwa14/collision/link_6_s.stl; visual mesh filename=../kuka_description/meshes/iiwa14/visual/link_6.stl
- link link_7: geometry collision mesh filename=../kuka_description/meshes/iiwa14/collision/link_7-MF-Touch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; visual mesh filename=../kuka_description/meshes/iiwa14/visual/link_7-MF-Touch-pn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
